Commit message: fixed some values

File: src/robotaksi_description/urdf/bee1.urdf.xacro (robot description, xacro)
@@ -33,4 +33,10 @@
     <origin xyz="0 0 ${govde_z_offset + govde_yukseklik/2}" rpy="0 0 0"/>
   </joint>
+  <link name="front_aks"/>
+  <joint name="front_aks_joint" type="fixed">
+    <parent link="base_footprint"/>
+    <child link="front_aks"/>
+    <origin xyz="0.96 0 0" rpy="0 0 0"/>
+  </joint>
   <xacro:macro name="tekerlek" params="ad x_ofset y_ofset">
     <link name="${ad}">
@@ -60,8 +66,8 @@
     </joint>
   </xacro:macro>
-  <xacro:tekerlek ad="tekerlek_on_sol"   x_ofset="${dingil_mesafesi/2}"  y_ofset="${govde_genislik/2 + 0.08}"/>
-  <xacro:tekerlek ad="tekerlek_on_sag"   x_ofset="${dingil_mesafesi/2}"  y_ofset="-${govde_genislik/2 + 0.08}"/>
-  <xacro:tekerlek ad="tekerlek_arka_sol" x_ofset="-${dingil_mesafesi/2}" y_ofset="${govde_genislik/2 + 0.08}"/>
-  <xacro:tekerlek ad="tekerlek_arka_sag" x_ofset="-${dingil_mesafesi/2}" y_ofset="-${govde_genislik/2 + 0.08}"/>
+  <xacro:tekerlek ad="tekerlek_on_sol"   x_ofset="0.96"  y_ofset="0.443"/>
+  <xacro:tekerlek ad="tekerlek_on_sag"   x_ofset="0.96"  y_ofset="-0.443"/>
+  <xacro:tekerlek ad="tekerlek_arka_sol" x_ofset="-0.9" y_ofset="0.425"/>
+  <xacro:tekerlek ad="tekerlek_arka_sag" x_ofset="-0.9" y_ofset="-0.425"/>
   <link name="lidar_link">
     <visual>
@@ -71,7 +77,7 @@
   </link>
   <joint name="lidar_joint" type="fixed">
-    <parent link="base_link"/>
+    <parent link="front_aks"/>
     <child link="lidar_link"/>
-    <origin xyz="-0.177 0 ${govde_yukseklik/2 + 0.1}" rpy="0 0 0"/>
+    <origin xyz="-0.177 0 0.62" rpy="0 0 0"/>
   </joint>
   <link name="kamera_sag_link">
@@ -82,7 +88,7 @@
   </link>
   <joint name="kamera_sag_joint" type="fixed">
-    <parent link="base_link"/>
+    <parent link="front_aks"/>
     <child link="kamera_sag_link"/>
-    <origin xyz="0.620 -0.060 ${govde_yukseklik/2}" rpy="0 0 0"/>
+    <origin xyz="-0.205 0.06 0.685" rpy="0 0 0"/>
   </joint>
   <link name="kamera_sol_link">
@@ -93,7 +99,7 @@
   </link>
   <joint name="kamera_sol_joint" type="fixed">
-    <parent link="base_link"/>
+    <parent link="front_aks"/>
     <child link="kamera_sol_link"/>
-    <origin xyz="0.685 0.060 ${govde_yukseklik/2}" rpy="0 0 0"/>
+    <origin xyz="-0.205 -0.06 0.685" rpy="0 0 0"/>
   </joint>
   <link name="gps_imu_link">
@@ -104,7 +110,7 @@
   </link>
   <joint name="gps_imu_joint" type="fixed">
-    <parent link="base_link"/>
+    <parent link="front_aks"/>
     <child link="gps_imu_link"/>
-    <origin xyz="1.440 0 ${govde_yukseklik/2 + 0.1}" rpy="0 0 0"/>
+    <origin xyz="1.44 0 1.39" rpy="0 0 0"/>
   </joint>
   <gazebo>

Commit message: added kasa but joint xyz is wrong for now

File: src/robotaksi_description/urdf/bee1.urdf.xacro (robot description, xacro)
@@ -6,4 +6,7 @@
   <xacro:property name="govde_z_offset" value="0.45"/>   <xacro:property name="tekerlek_yaricap" value="0.25"/>
   <xacro:property name="tekerlek_genislik" value="0.18"/>
+  <xacro:property name="kasa_uzunluk" value="1.2"/>
+  <xacro:property name="kasa_genislik" value="${govde_genislik}"/>
+  <xacro:property name="kasa_yukseklik" value="1.2"/>
   <material name="beyaz"><color rgba="0.95 0.95 0.95 1"/></material>
   <material name="siyah"><color rgba="0.05 0.05 0.05 1"/></material>
@@ -27,4 +30,34 @@
     </inertial>
   </link>
+  <link name="kasa_link">
+    <visual>
+      <origin xyz="0 0 0" rpy="0 0 0"/>
+      <geometry>
+        <box size="${kasa_uzunluk} ${kasa_genislik} ${kasa_yukseklik}"/>
+      </geometry>
+      <material name="beyaz"/>
+    </visual>
+    <collision>
+      <origin xyz="0 0 0" rpy="0 0 0"/>
+      <geometry>
+        <box size="${kasa_uzunluk} ${kasa_genislik} ${kasa_yukseklik}"/>
+      </geometry>
+    </collision>
+    <inertial>
+      <mass value="40.0"/>
+      <inertia
+        ixx="${40.0 * (kasa_genislik * kasa_genislik + kasa_yukseklik * kasa_yukseklik) / 12.0}"
+        ixy="0"
+        ixz="0"
+        iyy="${40.0 * (kasa_uzunluk * kasa_uzunluk + kasa_yukseklik * kasa_yukseklik) / 12.0}"
+        iyz="0"
+        izz="${40.0 * (kasa_genislik * kasa_genislik + kasa_uzunluk * kasa_uzunluk) / 12.0}"/>
+    </inertial>
+  </link>
+  <joint name="kasa_joint" type="fixed">
+    <parent link="base_link"/>
+    <child link="kasa_link"/>
+    <origin xyz="-${(govde_uzunluk/2)-(kasa_uzunluk/2)} 0 ${(govde_yukseklik/2)+(kasa_yukseklik/2)-0.5}"/>
+  </joint>
   <link name="base_footprint"/>
   <joint name="base_footprint_joint" type="fixed">
@@ -134,4 +167,7 @@
     </plugin>
   </gazebo>
+  <gazebo reference="kasa_link">
+    <material>Gazebo/White</material>
+  </gazebo>
   <gazebo reference="lidar_link">
     <sensor name="lidar" type="ray">

Commit message: I can't see the caaar

File: src/robotaksi_description/urdf/bee1.urdf.xacro (robot description, xacro)
@@ -72,4 +72,34 @@
     <origin xyz="0.96 0 0" rpy="0 0 0"/>
   </joint>
+  <xacro:macro name="dikiz_aynasi" params="ad y_ofset">
+    <link name="${ad}">
+      <visual>
+        <origin xyz="0 0 0" rpy="0 0 0"/>
+        <geometry>
+          <box size="0.08 0.18 0.12"/>
+        </geometry>
+        <material name="siyah"/>
+      </visual>
+      <collision>
+        <origin xyz="0 0 0" rpy="0 0 0"/>
+        <geometry>
+          <box size="0.08 0.18 0.12"/>
+        </geometry>
+      </collision>
+      <inertial>
+        <mass value="1.0"/>  <inertia ixx="0.003" ixy="0" ixz="0" iyy="0.003" iyz="0" izz="0.003" />
+      </inertial>
+    </link>
+    <joint name="${ad}_joint" type="fixed">
+      <parent link="base_link"/>
+      <child link="${ad}"/>
+      <origin xyz="0.4 ${y_ofset * (govde_genislik / 2) + (0.18 / 2)} 0.3" rpy="0 0 0"/>
+    </joint>
+    <gazebo reference="${ad}">
+      <material>Gazebo/Black</material>
+    </gazebo>
+  </xacro:macro>
+  <xacro:dikiz_aynasi ad="dikiz_sol"   y_ofset="1.13" />
+  <xacro:dikiz_aynasi ad="dikiz_sag"   y_ofset="0.79" />
   <xacro:macro name="tekerlek" params="ad x_ofset y_ofset">
     <link name="${ad}">
@@ -125,4 +155,10 @@
     <origin xyz="-0.205 0.06 0.685" rpy="0 0 0"/>
   </joint>
+  <link name="kamera_sag_link_optical"/>
+  <joint name="kamera_sag_link_optical_joint">
+    <parent link="kamera_sag_link"/>
+    <child link="kamera_sag_link_optical"/>
+    <origin xyz="0 0 0" rpy="-1.5708 0 -1.5708"/>
+  </joint>
   <link name="kamera_sol_link">
     <visual>
@@ -135,4 +171,10 @@
     <child link="kamera_sol_link"/>
     <origin xyz="-0.205 -0.06 0.685" rpy="0 0 0"/>
+  </joint>
+  <link name="kamera_sol_link_optical"/>
+  <joint name="kamera_sol_link_optical_joint">
+    <parent link="kamera_sol_link"/>
+    <child link="kamera_sol_link_optical"/>
+    <origin xyz="0 0 0" rpy="-1.5708 0 -1.5708"/>
   </joint>
   <link name="gps_imu_link">

Commit message: cameras and gps/imu worksss

File: src/robotaksi_description/urdf/bee1.urdf.xacro (robot description, xacro)
@@ -27,5 +27,5 @@
     </collision>
     <inertial>
-      <mass value="760"/>  <inertia ixx="200" ixy="0" ixz="0" iyy="400" iyz="0" izz="400"/>
+      <mass value="760"/>  <inertia ixx="273.2" ixy="0" ixz="0" iyy="472.9" iyz="0" izz="467.5"/>
     </inertial>
   </link>
@@ -66,5 +66,10 @@
     <origin xyz="0 0 ${govde_z_offset + govde_yukseklik/2}" rpy="0 0 0"/>
   </joint>
-  <link name="front_aks"/>
+  <link name="front_aks">
+    <inertial>
+      <mass value="0.1"/>
+      <inertia ixx="0.001" ixy="0" ixz="0" iyy="0.001" iyz="0" izz="0.001"/>
+    </inertial>
+  </link>
   <joint name="front_aks_joint" type="fixed">
     <parent link="base_footprint"/>
@@ -101,5 +106,5 @@
   </xacro:macro>
   <xacro:dikiz_aynasi ad="dikiz_sol"   y_ofset="1.13" />
-  <xacro:dikiz_aynasi ad="dikiz_sag"   y_ofset="0.79" />
+  <xacro:dikiz_aynasi ad="dikiz_sag"   y_ofset="-1.13" />
   <xacro:macro name="tekerlek" params="ad x_ofset y_ofset">
     <link name="${ad}">
@@ -156,5 +161,5 @@
   </joint>
   <link name="kamera_sag_link_optical"/>
-  <joint name="kamera_sag_link_optical_joint">
+  <joint name="kamera_sag_link_optical_joint" type="fixed">
     <parent link="kamera_sag_link"/>
     <child link="kamera_sag_link_optical"/>
@@ -173,5 +178,5 @@
   </joint>
   <link name="kamera_sol_link_optical"/>
-  <joint name="kamera_sol_link_optical_joint">
+  <joint name="kamera_sol_link_optical_joint" type="fixed">
     <parent link="kamera_sol_link"/>
     <child link="kamera_sol_link_optical"/>
@@ -242,3 +247,53 @@
     </sensor>
   </gazebo>
+  <xacro:macro name="gazebo_kamera_sensor" params="referans_linki ad topic_adi">
+    <gazebo reference="${referans_linki}">
+      <sensor type="camera" name="sensor_${ad}">
+        <update_rate>30.0</update_rate>
+        <camera name="${ad}">
+          <horizontal_fov>1.92</horizontal_fov>
+          <image>
+            <width>1280</width>
+            <height>720</height>
+            <format>R8G8B8</format>
+          </image>
+          <clip><near>0.1</near><far>100.0</far></clip>
+        </camera>
+        <plugin name="${ad}_kamera_surucu" filename="libgazebo_ros_camera.so">
+          <ros>
+            <namespace>/</namespace>
+            <remapping>~/image_raw:=camera/${topic_adi}/image_raw</remapping>
+            <remapping>~/camera_info:=camera/${topic_adi}/camera_info</remapping>
+          </ros>
+          <frame_name>${referans_linki}_optical</frame_name>
+        </plugin>
+      </sensor>
+    </gazebo>
+  </xacro:macro>
+  <xacro:gazebo_kamera_sensor referans_linki="kamera_sol_link" ad="sol" topic_adi="left"/>
+  <xacro:gazebo_kamera_sensor referans_linki="kamera_sag_link" ad="sag" topic_adi="right"/>
+  <gazebo reference="gps_imu_link">
+    <sensor type="gps" name="gps_sensor">
+      <always_on>true</always_on>
+      <update_rate>10.0</update_rate>
+      <plugin name="gps_surucu" filename="libgazebo_ros_gps_sensor.so">
+        <ros>
+          <namespace>/</namespace>
+          <remapping>~/out:=gps/data</remapping>
+        </ros>
+        <frame_name>gps_imu_link</frame_name>
+      </plugin>
+    </sensor>
+    <sensor type="imu" name="gps_sensor">
+      <always_on>true</always_on>
+      <update_rate>100.0</update_rate>
+      <plugin name="imu_surucu" filename="libgazebo_ros_imu_sensor.so">
+        <ros>
+          <namespace>/</namespace>
+          <remapping>~/out:=imu/data</remapping>
+        </ros>
+        <frame_name>gps_imu_link</frame_name>
+      </plugin>
+    </sensor>
+  </gazebo>
 </robot>

Commit message: added limits

File: src/robotaksi_description/urdf/bee1.urdf.xacro (robot description, xacro)
@@ -138,4 +138,20 @@
   <xacro:tekerlek ad="tekerlek_arka_sol" x_ofset="-0.9" y_ofset="0.425"/>
   <xacro:tekerlek ad="tekerlek_arka_sag" x_ofset="-0.9" y_ofset="-0.425"/>
+  <link name="aks_on_sol"/>
+  <joint name="aks_on_sol_joint" type="revolute">
+      <parent link="base_footprint"/>
+      <child link="aks_on_sol"/>
+      <origin xyz="0.96 0.443 0.25" rpy="0 0 0"/>
+      <axis xyz="0 0 1"/>
+      <limit lower="-0.567" upper="0.567" effort="100.0" velocity="10.0"/>
+  </joint>
+  <link name="aks_on_sag"/>
+  <joint name="aks_on_sag_joint" type="revolute">
+      <parent link="base_footprint"/>
+      <child link="aks_on_sag"/>
+      <origin xyz="0.96 -0.443 0.25" rpy="0 0 0"/>
+      <axis xyz="0 0 1"/>
+      <limit lower="-0.567" upper="0.567" effort="100.0" velocity="10.0"/>
+  </joint>
   <link name="lidar_link">
     <visual>
@@ -297,3 +313,34 @@
     </sensor>
   </gazebo>
+  <gazebo>
+    <plugin name="ackerman" filename="libgazebo_ros_ackermann_drive.so">
+      <update_rate>100.0</update_rate>
+      <front_left_joint>tekerlek_on_sol_joint</front_left_joint>
+      <front_right_joint>tekerlek_on_sag_joint</front_right_joint>
+      <rear_left_joint>tekerlek_arka_sol_joint</rear_left_joint>
+      <rear_right_joint>tekerlek_arka_sag_joint</rear_right_joint>
+      <left_steering_joint>aks_on_sol_joint</left_steering_joint>
+      <right_steering_joint>aks_on_sag_joint</right_steering_joint>
+      <wheel_separation>0.886</wheel_separation>
+      <wheel_diameter>0.25</wheel_diameter>
+      <track_width>0.886</track_width>
+      <wheelbase>1.86</wheelbase>
+      <max_speed>8.33</max_speed>
+      <max_wheel_torque>80.0</max_wheel_torque>
+      <max_acceleration>2.5</max_acceleration>
+      <max_deceleration>-6.5</max_deceleration>
+      <max_steering_angle>0.567</max_steering_angle>
+      <steering_speed>10.0</steering_speed>
+      <ros>
+      <namespace>/</namespace>
+      <remapping>cmd_vel:=cmd_vel</remapping>
+      <remapping>odom:=odom</remapping>
+      </ros>
+      <publish_odom>true</publish_odom>
+      <publish_odom_tf>true</publish_odom_tf>
+      <publish_wheel_tf>true</publish_wheel_tf>
+      <odometry_frame>odom</odometry_frame>
+      <robot_base_frame>base_footprint</robot_base_frame>
+    </plugin>
+  </gazebo>
 </robot>

Commit message: Car is ready I think

File: src/robotaksi_description/urdf/bee1.urdf.xacro (robot description, xacro)
@@ -7,5 +7,5 @@
   <xacro:property name="tekerlek_genislik" value="0.18"/>
   <xacro:property name="kasa_uzunluk" value="1.2"/>
-  <xacro:property name="kasa_genislik" value="${govde_genislik}"/>
+  <xacro:property name="kasa_genislik" value="1.1"/>
   <xacro:property name="kasa_yukseklik" value="1.2"/>
   <material name="beyaz"><color rgba="0.95 0.95 0.95 1"/></material>
@@ -13,37 +13,62 @@
   <material name="kirmizi"><color rgba="0.8 0 0 1"/></material>
   <link name="base_link">
-    <visual>
+    <inertial>
+      <origin xyz="0 0 0" rpy="0 0 0" />
+      <mass value="294.0" /> <inertia
+        ixx="${(1/12) * 50.0 * (govde_genislik*govde_genislik + govde_yukseklik*govde_yukseklik)}" ixy="0.0" ixz="0.0"
+        iyy="${(1/12) * 50.0 * (govde_uzunluk*govde_uzunluk + govde_yukseklik*govde_yukseklik)}" iyz="0.0"
+        izz="${(1/12) * 50.0 * (govde_uzunluk*govde_uzunluk + govde_genislik*govde_genislik)}" />
+    </inertial>
+    <collision>
       <origin xyz="0 0 0" rpy="0 0 0"/>
       <geometry>
         <box size="${govde_uzunluk} ${govde_genislik} ${govde_yukseklik}"/>
       </geometry>
+    </collision>
+  </link>
+  <link name="arka_kabin_link">
+    <visual>
+      <origin xyz="0 0 0" rpy="0 0 0"/>
+      <geometry>
+        <box size="${4 * govde_uzunluk / 5} ${govde_genislik} ${govde_yukseklik}"/>
+      </geometry>
       <material name="beyaz"/>
     </visual>
+  </link>
+  <joint name="arka_kabin_joint" type="fixed">
+    <parent link="base_link"/>
+    <child link="arka_kabin_link"/>
+    <origin xyz="-${govde_uzunluk / 10} 0 0" rpy="0 0 0"/>
+  </joint>
+  <link name="on_kabin_link">
+    <visual>
+      <origin xyz="0 0 0" rpy="0 0 0"/>
+      <geometry>
+        <box size="${govde_uzunluk / 5} ${govde_genislik} ${2 * govde_yukseklik / 3}"/>
+      </geometry>
+      <material name="beyaz"/>
+    </visual>
+  </link>
+  <joint name="on_kabin_joint" type="fixed">
+    <parent link="base_link"/>
+    <child link="on_kabin_link"/>
+    <origin xyz="${4 * govde_uzunluk / 10} 0 -${govde_yukseklik / 6}" rpy="0 0 0"/>
+  </joint>
+  <link name="kasa_link">
+    <visual>
+      <origin xyz="0 0 0" rpy="0 0 0"/>
+      <geometry>
+        <box size="${kasa_uzunluk} ${kasa_genislik} ${kasa_yukseklik}"/>
+      </geometry>
+      <material name="beyaz"/>
+    </visual>
     <collision>
       <origin xyz="0 0 0" rpy="0 0 0"/>
       <geometry>
-        <box size="${govde_uzunluk} ${govde_genislik} ${govde_yukseklik}"/>
+        <box size="${kasa_uzunluk} ${kasa_genislik} ${kasa_yukseklik}"/>
       </geometry>
     </collision>
     <inertial>
-      <mass value="760"/>  <inertia ixx="273.2" ixy="0" ixz="0" iyy="472.9" iyz="0" izz="467.5"/>
-    </inertial>
-  </link>
-  <link name="kasa_link">
-    <visual>
-      <origin xyz="0 0 0" rpy="0 0 0"/>
-      <geometry>
-        <box size="${kasa_uzunluk} ${kasa_genislik} ${kasa_yukseklik}"/>
-      </geometry>
-      <material name="beyaz"/>
-    </visual>
-    <collision>
-      <origin xyz="0 0 0" rpy="0 0 0"/>
-      <geometry>
-        <box size="${kasa_uzunluk} ${kasa_genislik} ${kasa_yukseklik}"/>
-      </geometry>
-    </collision>
-    <inertial>
-      <mass value="40.0"/>
+      <mass value="406.0"/>
       <inertia
         ixx="${40.0 * (kasa_genislik * kasa_genislik + kasa_yukseklik * kasa_yukseklik) / 12.0}"
@@ -58,5 +83,5 @@
     <parent link="base_link"/>
     <child link="kasa_link"/>
-    <origin xyz="-${(govde_uzunluk/2)-(kasa_uzunluk/2)} 0 ${(govde_yukseklik/2)+(kasa_yukseklik/2)-0.5}"/>
+    <origin xyz="-0.875 0 0.4275"/>
   </joint>
   <link name="base_footprint"/>
@@ -82,5 +107,5 @@
         <origin xyz="0 0 0" rpy="0 0 0"/>
         <geometry>
-          <box size="0.08 0.18 0.12"/>
+          <box size="0.17 0.18 0.12"/>
         </geometry>
         <material name="siyah"/>
@@ -89,5 +114,5 @@
         <origin xyz="0 0 0" rpy="0 0 0"/>
         <geometry>
-          <box size="0.08 0.18 0.12"/>
+          <box size="0.17 0.18 0.12"/>
         </geometry>
       </collision>
@@ -99,5 +124,5 @@
       <parent link="base_link"/>
       <child link="${ad}"/>
-      <origin xyz="0.4 ${y_ofset * (govde_genislik / 2) + (0.18 / 2)} 0.3" rpy="0 0 0"/>
+      <origin xyz="0.6 ${y_ofset} 0" rpy="0 0 0"/>
     </joint>
     <gazebo reference="${ad}">
@@ -105,6 +130,6 @@
     </gazebo>
   </xacro:macro>
-  <xacro:dikiz_aynasi ad="dikiz_sol"   y_ofset="1.13" />
-  <xacro:dikiz_aynasi ad="dikiz_sag"   y_ofset="-1.13" />
+  <xacro:dikiz_aynasi ad="dikiz_sol"   y_ofset="0.615"/>
+  <xacro:dikiz_aynasi ad="dikiz_sag"   y_ofset="-0.615"/>
   <xacro:macro name="tekerlek" params="ad x_ofset y_ofset">
     <link name="${ad}">
@@ -229,4 +254,16 @@
       <publish_wheel_tf>true</publish_wheel_tf>
     </plugin>
+  </gazebo>
+  <gazebo reference="tekerlek_on_sol">
+    <material>Gazebo/Black</material>
+  </gazebo>
+  <gazebo reference="tekerlek_on_sag">
+    <material>Gazebo/Black</material>
+  </gazebo>
+  <gazebo reference="tekerlek_arka_sol">
+    <material>Gazebo/Black</material>
+  </gazebo>
+  <gazebo reference="tekerlek_arka_sag">
+    <material>Gazebo/Black</material>
   </gazebo>
   <gazebo reference="kasa_link">

Commit message: sensörler çalışıyor ancak kullanan bir birim olmadığı için bağlanmıyorlar, ackermann'da hata veriyor ama hata vermemesi lazım; noise sıkıntısını çözdüm

File: src/robotaksi_description/urdf/bee1.urdf.xacro (robot description, xacro)
@@ -165,7 +165,7 @@
   <link name="aks_on_sol"/>
   <joint name="aks_on_sol_joint" type="revolute">
-      <parent link="base_footprint"/>
+      <parent link="base_link"/>
       <child link="aks_on_sol"/>
-      <origin xyz="0.96 0.443 0.25" rpy="0 0 0"/>
+      <origin xyz="0.96 -0.443 0.25" rpy="0 0 0"/>
       <axis xyz="0 0 1"/>
       <limit lower="-0.567" upper="0.567" effort="100.0" velocity="10.0"/>
@@ -173,7 +173,7 @@
   <link name="aks_on_sag"/>
   <joint name="aks_on_sag_joint" type="revolute">
-      <parent link="base_footprint"/>
+      <parent link="base_link"/>
       <child link="aks_on_sag"/>
-      <origin xyz="0.96 -0.443 0.25" rpy="0 0 0"/>
+      <origin xyz="0.96 0.443 0.25" rpy="0 0 0"/>
       <axis xyz="0 0 1"/>
       <limit lower="-0.567" upper="0.567" effort="100.0" velocity="10.0"/>
@@ -288,4 +288,9 @@
           <max>100.0</max>
           <resolution>0.03</resolution>
+          <noise>
+            <type>gaussian</type>
+            <mean>0.0</mean>
+            <stddev>0.01</stddev>
+          </noise>
         </range>
       </ray>
@@ -312,4 +317,9 @@
           </image>
           <clip><near>0.1</near><far>100.0</far></clip>
+          <noise>
+            <type>gaussian</type>
+            <mean>0.0</mean>
+            <stddev>0.007</stddev>
+          </noise>
         </camera>
         <plugin name="${ad}_kamera_surucu" filename="libgazebo_ros_camera.so">
@@ -341,4 +351,16 @@
       <always_on>true</always_on>
       <update_rate>100.0</update_rate>
+      <imu>
+        <angular_velocity>
+          <x><noise type="gaussian"><mean>0.0</mean><stddev>0.0</stddev></noise></x>
+          <y><noise type="gaussian"><mean>0.0</mean><stddev>0.0</stddev></noise></y>
+          <z><noise type="gaussian"><mean>0.0</mean><stddev>0.0</stddev></noise></z>
+        </angular_velocity>
+        <linear_acceleration>
+          <x><noise type="gaussian"><mean>0.0</mean><stddev>0.0</stddev></noise></x>
+          <y><noise type="gaussian"><mean>0.0</mean><stddev>0.0</stddev></noise></y>
+          <z><noise type="gaussian"><mean>0.0</mean><stddev>0.0</stddev></noise></z>
+        </linear_acceleration>
+      </imu>
       <plugin name="imu_surucu" filename="libgazebo_ros_imu_sensor.so">
         <ros>
@@ -353,10 +375,10 @@
     <plugin name="ackerman" filename="libgazebo_ros_ackermann_drive.so">
       <update_rate>100.0</update_rate>
+      <left_steering_joint>aks_on_sol_joint</left_steering_joint>
+      <right_steering_joint>aks_on_sag_joint</right_steering_joint>
       <front_left_joint>tekerlek_on_sol_joint</front_left_joint>
       <front_right_joint>tekerlek_on_sag_joint</front_right_joint>
       <rear_left_joint>tekerlek_arka_sol_joint</rear_left_joint>
       <rear_right_joint>tekerlek_arka_sag_joint</rear_right_joint>
-      <left_steering_joint>aks_on_sol_joint</left_steering_joint>
-      <right_steering_joint>aks_on_sag_joint</right_steering_joint>
       <wheel_separation>0.886</wheel_separation>
       <wheel_diameter>0.25</wheel_diameter>
@@ -370,7 +392,7 @@
       <steering_speed>10.0</steering_speed>
       <ros>
-      <namespace>/</namespace>
-      <remapping>cmd_vel:=cmd_vel</remapping>
-      <remapping>odom:=odom</remapping>
+        <namespace>/</namespace>
+        <remapping>/cmd_vel:=/cmd_vel</remapping>
+        <remapping>/odom:=/odom</remapping>
       </ros>
       <publish_odom>true</publish_odom>

Commit message: feat: trying to make the obstacle detection happen

File: src/robotaksi_description/urdf/bee1.urdf.xacro (robot description, xacro)
@@ -111,12 +111,8 @@
         <material name="siyah"/>
       </visual>
-      <collision>
-        <origin xyz="0 0 0" rpy="0 0 0"/>
-        <geometry>
-          <box size="0.17 0.18 0.12"/>
-        </geometry>
-      </collision>
+      <!-- collision removed: mirrors don't need physics collision -->
       <inertial>
-        <mass value="1.0"/>  <inertia ixx="0.003" ixy="0" ixz="0" iyy="0.003" iyz="0" izz="0.003" />
+        <mass value="1.0"/>
+        <inertia ixx="0.003" ixy="0" ixz="0" iyy="0.003" iyz="0" izz="0.003" />
       </inertial>
     </link>
@@ -188,5 +184,5 @@
     <parent link="front_aks"/>
     <child link="lidar_link"/>
-    <origin xyz="-0.177 0 0.62" rpy="0 0 0"/>
+    <origin xyz="-0.177 0 1.5" rpy="0 0 0"/>
   </joint>
   <link name="kamera_sag_link">
@@ -290,5 +286,5 @@
         </scan>
         <range>
-          <min>0.1</min>
+          <min>0.7</min>
           <max>100.0</max>
           <resolution>0.03</resolution>
