Commit message: feat: lastest changes

File: src/robotaksi_description/urdf/bee1.urdf.xacro (robot description, xacro)
@@ -1,8 +1,10 @@
 <?xml version="1.0"?>
 <robot name="bee1" xmlns:xacro="http://www.ros.org/wiki/xacro">
-  <xacro:property name="govde_uzunluk" value="2.740"/>   <xacro:property name="govde_genislik" value="1.060"/>
+  <xacro:property name="govde_uzunluk" value="2.740"/>
+  <xacro:property name="govde_genislik" value="1.060"/>
   <xacro:property name="govde_yukseklik" value="1.785"/>
   <xacro:property name="dingil_mesafesi" value="1.860"/>
-  <xacro:property name="govde_z_offset" value="0.45"/>   <xacro:property name="tekerlek_yaricap" value="0.25"/>
+  <xacro:property name="govde_z_offset" value="0.45"/>
+  <xacro:property name="tekerlek_yaricap" value="0.25"/>
   <xacro:property name="tekerlek_genislik" value="0.18"/>
   <xacro:property name="kasa_uzunluk" value="1.2"/>
@@ -13,7 +15,15 @@
   <material name="kirmizi"><color rgba="0.8 0 0 1"/></material>
   <link name="base_link">
+    <visual>
+      <origin xyz="0 0 0" rpy="0 0 0"/>
+      <geometry>
+        <box size="${govde_uzunluk} ${govde_genislik} ${govde_yukseklik}"/>
+      </geometry>
+      <material name="beyaz"/>
+    </visual>
     <inertial>
       <origin xyz="0 0 0" rpy="0 0 0" />
-      <mass value="294.0" /> <inertia
+      <mass value="294.0" />
+      <inertia
         ixx="${(1/12) * 50.0 * (govde_genislik*govde_genislik + govde_yukseklik*govde_yukseklik)}" ixy="0.0" ixz="0.0"
         iyy="${(1/12) * 50.0 * (govde_uzunluk*govde_uzunluk + govde_yukseklik*govde_yukseklik)}" iyz="0.0"
@@ -73,6 +83,5 @@
       <inertia
         ixx="${40.0 * (kasa_genislik * kasa_genislik + kasa_yukseklik * kasa_yukseklik) / 12.0}"
-        ixy="0"
-        ixz="0"
+        ixy="0" ixz="0"
         iyy="${40.0 * (kasa_uzunluk * kasa_uzunluk + kasa_yukseklik * kasa_yukseklik) / 12.0}"
         iyz="0"
@@ -111,5 +120,4 @@
         <material name="siyah"/>
       </visual>
-      <!-- collision removed: mirrors don't need physics collision -->
       <inertial>
         <mass value="1.0"/>
@@ -126,6 +134,6 @@
     </gazebo>
   </xacro:macro>
-  <xacro:dikiz_aynasi ad="dikiz_sol"   y_ofset="0.615"/>
-  <xacro:dikiz_aynasi ad="dikiz_sag"   y_ofset="-0.615"/>
+  <xacro:dikiz_aynasi ad="dikiz_sol" y_ofset="0.615"/>
+  <xacro:dikiz_aynasi ad="dikiz_sag" y_ofset="-0.615"/>
   <xacro:macro name="tekerlek" params="ad x_ofset y_ofset">
     <link name="${ad}">
@@ -157,21 +165,21 @@
   <xacro:tekerlek ad="tekerlek_on_sol"   x_ofset="0.96"  y_ofset="0.443"/>
   <xacro:tekerlek ad="tekerlek_on_sag"   x_ofset="0.96"  y_ofset="-0.443"/>
-  <xacro:tekerlek ad="tekerlek_arka_sol" x_ofset="-0.9" y_ofset="0.425"/>
-  <xacro:tekerlek ad="tekerlek_arka_sag" x_ofset="-0.9" y_ofset="-0.425"/>
+  <xacro:tekerlek ad="tekerlek_arka_sol" x_ofset="-0.9"  y_ofset="0.425"/>
+  <xacro:tekerlek ad="tekerlek_arka_sag" x_ofset="-0.9"  y_ofset="-0.425"/>
   <link name="aks_on_sol"/>
   <joint name="aks_on_sol_joint" type="revolute">
-      <parent link="base_link"/>
-      <child link="aks_on_sol"/>
-      <origin xyz="0.96 -0.443 0.25" rpy="0 0 0"/>
-      <axis xyz="0 0 1"/>
-      <limit lower="-0.567" upper="0.567" effort="100.0" velocity="10.0"/>
+    <parent link="base_link"/>
+    <child link="aks_on_sol"/>
+    <origin xyz="0.96 -0.443 0.25" rpy="0 0 0"/>
+    <axis xyz="0 0 1"/>
+    <limit lower="-0.567" upper="0.567" effort="100.0" velocity="10.0"/>
   </joint>
   <link name="aks_on_sag"/>
   <joint name="aks_on_sag_joint" type="revolute">
-      <parent link="base_link"/>
-      <child link="aks_on_sag"/>
-      <origin xyz="0.96 0.443 0.25" rpy="0 0 0"/>
-      <axis xyz="0 0 1"/>
-      <limit lower="-0.567" upper="0.567" effort="100.0" velocity="10.0"/>
+    <parent link="base_link"/>
+    <child link="aks_on_sag"/>
+    <origin xyz="0.96 0.443 0.25" rpy="0 0 0"/>
+    <axis xyz="0 0 1"/>
+    <limit lower="-0.567" upper="0.567" effort="100.0" velocity="10.0"/>
   </joint>
   <link name="lidar_link">
@@ -184,5 +192,5 @@
     <parent link="front_aks"/>
     <child link="lidar_link"/>
-    <origin xyz="-0.177 0 1.5" rpy="0 0 0"/>
+    <origin xyz="-0.177 0 0.62" rpy="0 0 0"/>
   </joint>
   <link name="kamera_sag_link">
@@ -243,5 +251,5 @@
       <max_speed>8.33</max_speed>
       <max_acceleration>2.5</max_acceleration>
-      <max_deceleration>-6.5</max_deceleration>
+      <max_deceleration>6.5</max_deceleration>
       <max_steering_angle>0.567</max_steering_angle>
       <steering_speed>10.0</steering_speed>
@@ -256,19 +264,9 @@
     </plugin>
   </gazebo>
-  <gazebo reference="tekerlek_on_sol">
-    <material>Gazebo/Black</material>
-  </gazebo>
-  <gazebo reference="tekerlek_on_sag">
-    <material>Gazebo/Black</material>
-  </gazebo>
-  <gazebo reference="tekerlek_arka_sol">
-    <material>Gazebo/Black</material>
-  </gazebo>
-  <gazebo reference="tekerlek_arka_sag">
-    <material>Gazebo/Black</material>
-  </gazebo>
-  <gazebo reference="kasa_link">
-    <material>Gazebo/White</material>
-  </gazebo>
+  <gazebo reference="tekerlek_on_sol"><material>Gazebo/Black</material></gazebo>
+  <gazebo reference="tekerlek_on_sag"><material>Gazebo/Black</material></gazebo>
+  <gazebo reference="tekerlek_arka_sol"><material>Gazebo/Black</material></gazebo>
+  <gazebo reference="tekerlek_arka_sag"><material>Gazebo/Black</material></gazebo>
+  <gazebo reference="kasa_link"><material>Gazebo/White</material></gazebo>
   <gazebo reference="lidar_link">
     <sensor name="lidar" type="ray">
@@ -349,5 +347,6 @@
       </plugin>
     </sensor>
-    <sensor type="imu" name="gps_sensor">
+    <!-- FIX 3: renamed from "gps_sensor" to "imu_sensor" to avoid name collision -->
+    <sensor type="imu" name="imu_sensor">
       <always_on>true</always_on>
       <update_rate>100.0</update_rate>
